File: Bafang_LCD_SW102/SW102_nRF51x22.sch (EAGLE design)
At the start: 24 parts, among them Q1 BSS123, Q2 BSS123, U1 NRF51X22_QFQF, X1 16MHz

Commit message: Updated naming to reflect real world names.
Parts:
- removed C1, C2: (no value), Nordic_nRF:CAPACITOR_0402_N
- removed C7: 4.7µF, Nordic_nRF:CAPACITOR_0603_N
- removed R3: 1k, rcl:R-EU_R0603
- added .R1: 10k, rcl:R-EU_R0603
- added .R25: 300k, rcl:R-EU_R0603
- added C14: 1.0pF, Nordic_nRF:CAPACITOR_0402_N
- added C18: 47nF, Nordic_nRF:CAPACITOR_0402_N
- added C23: 100nF, Nordic_nRF:CAPACITOR_0402_N
- C10: value 47nF -> 100nF
- C11: value 100nF -> 4.7µF; device Nordic_nRF:CAPACITOR_0402_N -> Nordic_nRF:CAPACITOR_0603_N
- C12: value 100nF -> 1.0nF
- C4: value 1.0pF -> 100nF
- C8: value 100nF -> (none)
- C9: value 1.0nF -> (none)
- R1: value 10k -> 1k
- R4: value 300k -> 10k
- renumbered C3 to C19, C5 to C13, C6 to C15, L1 to L4, L2 to L5, Q1 to .Q1, Q2 to .Q2, R2 to .R2, R5 to .R24, X1 to Y1
Connections:
- net +3V3: now also .R1.1, C12.1, C23.1, R4.2; no longer C7.1, C9.1, R1.1
- net BAT+_ADC: now also R1.2; no longer R3.2
- net GND: now also C14.2, C18.2, C23.2; no longer C1.2, C2.2, C7.2
- net LCD_RST: now also R4.1
- net N$10: now also C14.1; no longer C4.1
- net N$3: now also C8.1; no longer C1.1
- net N$4: now also .R25.1, C4.1, R1.1; no longer C12.1, R3.1, R4.1
- net N$5: now also C18.1; no longer C10.1
- net N$6: now also C10.1; no longer C8.1
- net UART_RX: now also .R1.2; no longer R1.2
- net VCC: now also .R25.2; no longer R4.2
- net X1: now also C9.1; no longer C2.1
Other:
- moved on the sheet: C10, C11, C12, C4, C8, C9, R1, R4

Commit message: Minor changes
Parts:
- .R1, .R2, R4: value 10k -> (none)
- C4: value 100nF -> (none)
Other:
- note added: "Bidirectional Level Shifter (on PowerBoard) Downstream pullup resistors are mandatory!"
- note removed: "Bidirectional Level Shifter (on PowerBoard)"
- moved on the sheet: .R1, .R2
Changed lines of the file:
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@@
 <part name=".Q1" library="transistor-small-signal" library_urn="urn:adsk.eagle:library:401" deviceset="BSS123" device="" package3d_urn="urn:adsk.eagle:package:28738/2"/>
 <part name=".Q2" library="transistor-small-signal" library_urn="urn:adsk.eagle:library:401" deviceset="BSS123" device="" package3d_urn="urn:adsk.eagle:package:28738/2"/>
-<part name=".R2" library="rcl" library_urn="urn:adsk.eagle:library:334" deviceset="R-EU_" device="R0603" package3d_urn="urn:adsk.eagle:package:23555/3" value="10k"/>
+<part name=".R2" library="rcl" library_urn="urn:adsk.eagle:library:334" deviceset="R-EU_" device="R0603" package3d_urn="urn:adsk.eagle:package:23555/3"/>
 <part name="+3V1" library="supply1" library_urn="urn:adsk.eagle:library:371" deviceset="+3V3" device=""/>
 <part name="+3V2" library="supply1" library_urn="urn:adsk.eagle:library:371" deviceset="+3V3" device=""/>
@@
 <part name="+3V5" library="supply1" library_urn="urn:adsk.eagle:library:371" deviceset="+3V3" device=""/>
 <part name="R1" library="rcl" library_urn="urn:adsk.eagle:library:334" deviceset="R-EU_" device="R0603" package3d_urn="urn:adsk.eagle:package:23555/3" value="1k"/>
-<part name="C4" library="Nordic_nRF" deviceset="CAPACITOR" device="_0402_N" value="100nF"/>
+<part name="C4" library="Nordic_nRF" deviceset="CAPACITOR" device="_0402_N"/>
 <part name="GND4" library="supply1" deviceset="GND" device=""/>
 <part name=".R25" library="rcl" library_urn="urn:adsk.eagle:library:334" deviceset="R-EU_" device="R0603" package3d_urn="urn:adsk.eagle:package:23555/3" value="300k"/>
@@
 <part name="GND9" library="supply1" deviceset="GND" device=""/>
 <part name="P+1" library="supply1" library_urn="urn:adsk.eagle:library:371" deviceset="VCC" device=""/>
-<part name=".R1" library="rcl" library_urn="urn:adsk.eagle:library:334" deviceset="R-EU_" device="R0603" package3d_urn="urn:adsk.eagle:package:23555/3" value="10k"/>
-<part name="R4" library="rcl" library_urn="urn:adsk.eagle:library:334" deviceset="R-EU_" device="R0603" package3d_urn="urn:adsk.eagle:package:23555/3" value="10k"/>
+<part name=".R1" library="rcl" library_urn="urn:adsk.eagle:library:334" deviceset="R-EU_" device="R0603" package3d_urn="urn:adsk.eagle:package:23555/3"/>
+<part name="R4" library="rcl" library_urn="urn:adsk.eagle:library:334" deviceset="R-EU_" device="R0603" package3d_urn="urn:adsk.eagle:package:23555/3"/>
 <part name="+3V6" library="supply1" library_urn="urn:adsk.eagle:library:371" deviceset="+3V3" device=""/>
 </parts>
@@
 <sheet>
 <plain>
-<text x="7.62" y="109.22" size="1.778" layer="91">Bidirectional Level Shifter (on PowerBoard)</text>
+<text x="7.62" y="106.68" size="1.778" layer="91">Bidirectional Level Shifter (on PowerBoard)
+Downstream pullup resistors are mandatory!</text>
 <text x="142.24" y="144.78" size="1.6764" layer="91">Function of Power Switch (PS):
 + PS turns on power as long as pressed.
@@
 <attribute name="NAME" x="43.18" y="144.78" size="1.778" layer="95" rot="MR270"/>
 </instance>
-<instance part=".R2" gate="G$1" x="50.8" y="154.94" smashed="yes" rot="R270">
-<attribute name="NAME" x="52.2986" y="158.75" size="1.778" layer="95" rot="R270"/>
-<attribute name="VALUE" x="47.498" y="158.75" size="1.778" layer="96" rot="R270"/>
-</instance>
-<instance part="+3V1" gate="G$1" x="50.8" y="167.64" smashed="yes">
-<attribute name="VALUE" x="48.26" y="162.56" size="1.778" layer="96" rot="R90"/>
-</instance>
-<instance part="+3V2" gate="G$1" x="50.8" y="139.7" smashed="yes">
-<attribute name="VALUE" x="48.26" y="134.62" size="1.778" layer="96" rot="R90"/>
+<instance part=".R2" gate="G$1" x="50.8" y="152.4" smashed="yes" rot="R270">
+<attribute name="NAME" x="52.2986" y="156.21" size="1.778" layer="95" rot="R270"/>
+<attribute name="VALUE" x="47.498" y="156.21" size="1.778" layer="96" rot="R270"/>
+</instance>
+<instance part="+3V1" gate="G$1" x="50.8" y="165.1" smashed="yes">
+<attribute name="VALUE" x="48.26" y="160.02" size="1.778" layer="96" rot="R90"/>
+</instance>
+<instance part="+3V2" gate="G$1" x="50.8" y="137.16" smashed="yes">
+<attribute name="VALUE" x="48.26" y="132.08" size="1.778" layer="96" rot="R90"/>
 </instance>
 <instance part="+3V3" gate="G$1" x="81.28" y="96.52" smashed="yes">
@@
 <attribute name="VALUE" x="15.24" y="71.12" size="1.778" layer="96" rot="R90"/>
 </instance>
-<instance part=".R1" gate="G$1" x="50.8" y="127" smashed="yes" rot="R270">
-<attribute name="NAME" x="52.2986" y="130.81" size="1.778" layer="95" rot="R270"/>
-<attribute name="VALUE" x="47.498" y="130.81" size="1.778" layer="96" rot="R270"/>
+<instance part=".R1" gate="G$1" x="50.8" y="124.46" smashed="yes" rot="R270">
+<attribute name="NAME" x="52.2986" y="128.27" size="1.778" layer="95" rot="R270"/>
+<attribute name="VALUE" x="47.498" y="128.27" size="1.778" layer="96" rot="R270"/>
 </instance>
 <instance part="R4" gate="G$1" x="71.12" y="86.36" smashed="yes" rot="R90">
@@
 <pinref part=".R2" gate="G$1" pin="2"/>
 <wire x1="48.26" y1="147.32" x2="50.8" y2="147.32" width="0.1524" layer="91"/>
-<wire x1="50.8" y1="147.32" x2="50.8" y2="149.86" width="0.1524" layer="91"/>
 <wire x1="50.8" y1="147.32" x2="71.12" y2="147.32" width="0.1524" layer="91" style="shortdash"/>
 <junction x="50.8" y="147.32"/>
@@
 <pinref part=".R1" gate="G$1" pin="2"/>
 <wire x1="48.26" y1="119.38" x2="50.8" y2="119.38" width="0.1524" layer="91"/>
-<wire x1="50.8" y1="119.38" x2="50.8" y2="121.92" width="0.1524" layer="91"/>
 <wire x1="50.8" y1="119.38" x2="71.12" y2="119.38" width="0.1524" layer="91" style="shortdash"/>
 <junction x="50.8" y="119.38"/>
@@
 <pinref part=".R2" gate="G$1" pin="1"/>
 <pinref part=".Q2" gate="G$1" pin="G"/>
-<wire x1="50.8" y1="160.02" x2="45.72" y2="160.02" width="0.1524" layer="91"/>
-<wire x1="45.72" y1="160.02" x2="45.72" y2="152.4" width="0.1524" layer="91"/>
+<wire x1="50.8" y1="157.48" x2="45.72" y2="157.48" width="0.1524" layer="91"/>
+<wire x1="45.72" y1="157.48" x2="45.72" y2="152.4" width="0.1524" layer="91"/>
 <pinref part="+3V1" gate="G$1" pin="+3V3"/>
-<wire x1="50.8" y1="165.1" x2="50.8" y2="160.02" width="0.1524" layer="91"/>
-<junction x="50.8" y="160.02"/>
+<wire x1="50.8" y1="162.56" x2="50.8" y2="157.48" width="0.1524" layer="91"/>
+<junction x="50.8" y="157.48"/>
 </segment>
 <segment>
 <pinref part=".R1" gate="G$1" pin="1"/>
 <pinref part=".Q1" gate="G$1" pin="G"/>
-<wire x1="50.8" y1="132.08" x2="45.72" y2="132.08" width="0.1524" layer="91"/>
-<wire x1="45.72" y1="132.08" x2="45.72" y2="124.46" width="0.1524" layer="91"/>
+<wire x1="50.8" y1="129.54" x2="45.72" y2="129.54" width="0.1524" layer="91"/>
+<wire x1="45.72" y1="129.54" x2="45.72" y2="124.46" width="0.1524" layer="91"/>
 <pinref part="+3V2" gate="G$1" pin="+3V3"/>
-<wire x1="50.8" y1="137.16" x2="50.8" y2="132.08" width="0.1524" layer="91"/>
-<junction x="50.8" y="132.08"/>
-</segment>
-<segment>
+<wire x1="50.8" y1="134.62" x2="50.8" y2="129.54" width="0.1524" layer="91"/>
+<junction x="50.8" y="129.54"/>
+</segment>
+<segment>
